Commit message: [urdf/freddy_base] Added robot name namespace for the laser scanners

File: urdf/freddy_base.urdf.xacro (robot description, xacro)
@@ -2,4 +2,5 @@
 <robot xmlns:xacro="http://www.ros.org/wiki/xacro">
     <!-- simplified box collision geometry for base -->
+    <xacro:property name="robot_name" value="freddy"/>
     <xacro:property name="base_size_x" value="0.635"/>
     <xacro:property name="base_size_y" value="0.582"/>
@@ -90,9 +91,9 @@
         <!-- HOKUYO LASER -->
         <xacro:hokuyo name="base_laser_front" parent="${name}_link"
-                           topic="base_scan_front" use_gpu="${use_gpu_2d_laser}">
+                           topic="/${robot_name}/base_scan_front" use_gpu="${use_gpu_2d_laser}">
             <origin xyz="0.26 -0.24 0.25" rpy="${pi} 0 ${-pi/4}"/>
         </xacro:hokuyo>
         <xacro:hokuyo name="base_laser_back" parent="${name}_link"
-                           topic="base_scan_back" use_gpu="${use_gpu_2d_laser}">
+                           topic="/${robot_name}/base_scan_back" use_gpu="${use_gpu_2d_laser}">
             <origin xyz="-0.26 0.24 0.25" rpy="${pi} 0 ${3*pi/4}"/>
         </xacro:hokuyo>

Commit message: [urdf/freddy_base] Added torso box

File: urdf/freddy_base.urdf.xacro (robot description, xacro)
@@ -3,4 +3,5 @@
     <!-- simplified box collision geometry for base -->
     <xacro:property name="robot_name" value="freddy"/>
+    <!-- base parameters -->
     <xacro:property name="base_size_x" value="0.635"/>
     <xacro:property name="base_size_y" value="0.582"/>
@@ -11,4 +12,9 @@
     <xacro:property name="base_size_z" value="${base_size_z_bottom + laser_slit_height + base_size_z_top}"/>
     <xacro:property name="base_mass" value="40.0"/>
+    <!-- torso parameters -->
+    <xacro:property name="torso_height" value="0.3"/>
+    <xacro:property name="torso_width" value="0.4"/>
+    <xacro:property name="torso_thickness" value="0.19"/>
+    <xacro:property name="torso_back_offset" value="0.02"/>
     <xacro:include filename="$(find freddy_description)/urdf/sensors/hokuyo.urdf.xacro" />
     <xacro:include filename="$(find freddy_description)/urdf/kelo_wheel.urdf.xacro" />
@@ -52,8 +58,29 @@
                 <material name="DarkGrey"/>
             </visual>
+            <visual>
+                <origin xyz="${-base_size_x/2 + torso_back_offset + torso_thickness/2} 0 ${wheel_slit_height + base_size_z + torso_height/2}" rpy="0 0 0"/>
+                <geometry>
+                    <box size="${torso_thickness} ${torso_width} ${torso_height}" />
+                </geometry>
+                <material name="DarkGrey"/>
+            </visual>
+            <!-- base collisions -->
             <collision>
                 <origin xyz="0 0 ${wheel_slit_height + base_size_z_bottom/2}" rpy="0 0 0.0"/>
                 <geometry>
                     <box size="${base_size_x} ${base_size_y} ${base_size_z_bottom}" />
+                </geometry>
+            </collision>
+            <collision>
+                <origin xyz="0 0 ${wheel_slit_height + base_size_z_bottom + laser_slit_height + base_size_z_top/2}" rpy="0 0 0.0"/>
+                <geometry>
+                    <box size="${base_size_x} ${base_size_y} ${base_size_z_top}" />
+                </geometry>
+            </collision>
+            <!-- torso collision -->
+            <collision>
+                <origin xyz="${-base_size_x/2 + torso_back_offset + torso_thickness/2} 0 ${wheel_slit_height + base_size_z + torso_height/2}" rpy="0 0 0"/>
+                <geometry>
+                    <box size="${torso_thickness} ${torso_width} ${torso_height}" />
                 </geometry>
             </collision>
