Commit message: Split the URDF into base and torso
freddy_description is now just merging the two.

The descriptions of the base and torso are in separate packages
freddy_base_description and freddy_torso_description.

The torso description is still incomplete (the arms haven't been added).

File: freddy_base_description/urdf/freddy_base.urdf.xacro (robot description, xacro)
@@ -3,5 +3,4 @@
     <!-- simplified box collision geometry for base -->
     <xacro:property name="robot_name" value="freddy"/>
-    <!-- base parameters -->
     <xacro:property name="base_size_x" value="0.635"/>
     <xacro:property name="base_size_y" value="0.582"/>
@@ -12,11 +11,6 @@
     <xacro:property name="base_size_z" value="${base_size_z_bottom + laser_slit_height + base_size_z_top}"/>
     <xacro:property name="base_mass" value="40.0"/>
-    <!-- torso parameters -->
-    <xacro:property name="torso_height" value="0.3"/>
-    <xacro:property name="torso_width" value="0.4"/>
-    <xacro:property name="torso_thickness" value="0.19"/>
-    <xacro:property name="torso_back_offset" value="0.02"/>
-    <xacro:include filename="$(find freddy_description)/urdf/sensors/hokuyo.urdf.xacro" />
-    <xacro:include filename="$(find freddy_description)/urdf/kelo_wheel.urdf.xacro" />
+    <xacro:include filename="$(find freddy_base_description)/urdf/sensors/hokuyo.urdf.xacro" />
+    <xacro:include filename="$(find freddy_base_description)/urdf/kelo_wheel.urdf.xacro" />
     <xacro:macro name="freddy_base" params="name parent *origin use_gpu_2d_laser:=true">
         <!-- HOLONOMIC DRIVE PLUGIN -->
@@ -30,5 +24,5 @@
             </plugin>
         </gazebo>
-        <!-- BODY -->
+        <!-- BASE -->
         <joint name="${name}_joint" type="fixed">
             <xacro:insert_block name="origin" />
@@ -58,12 +52,5 @@
                 <material name="DarkGrey"/>
             </visual>
-            <visual>
-                <origin xyz="${-base_size_x/2 + torso_back_offset + torso_thickness/2} 0 ${wheel_slit_height + base_size_z + torso_height/2}" rpy="0 0 0"/>
-                <geometry>
-                    <box size="${torso_thickness} ${torso_width} ${torso_height}" />
-                </geometry>
-                <material name="DarkGrey"/>
-            </visual>
-            <!-- base collisions -->
+            <!-- base bottom collisions -->
             <collision>
                 <origin xyz="0 0 ${wheel_slit_height + base_size_z_bottom/2}" rpy="0 0 0.0"/>
@@ -72,15 +59,9 @@
                 </geometry>
             </collision>
+            <!-- base top collisions -->
             <collision>
                 <origin xyz="0 0 ${wheel_slit_height + base_size_z_bottom + laser_slit_height + base_size_z_top/2}" rpy="0 0 0.0"/>
                 <geometry>
                     <box size="${base_size_x} ${base_size_y} ${base_size_z_top}" />
-                </geometry>
-            </collision>
-            <!-- torso collision -->
-            <collision>
-                <origin xyz="${-base_size_x/2 + torso_back_offset + torso_thickness/2} 0 ${wheel_slit_height + base_size_z + torso_height/2}" rpy="0 0 0"/>
-                <geometry>
-                    <box size="${torso_thickness} ${torso_width} ${torso_height}" />
                 </geometry>
             </collision>

File: freddy_base_description/urdf/kelo_wheel.urdf.xacro (robot description, xacro)
@@ -4,5 +4,5 @@
     <xacro:property name="wheel_mass" value="1.0" />
     <xacro:property name="inertia_wheels" value="0.001" />
-    <xacro:include filename="$(find freddy_description)/urdf/common.xacro" />
+    <xacro:include filename="$(find freddy_base_description)/urdf/common.xacro" />
     <xacro:macro name="kelo_wheel" params="name parent *origin material_name">
         <joint name="${name}_joint" type="fixed">
